Commit message: Last modifications

File: MB_robot/myrabot_arm_model/urdf/brazo-macros.xacro (robot description, xacro)
@@ -113,5 +113,5 @@
  <transmission type="pr2_mechanism_model/SimpleTransmission" name="base_trans">
     <actuator name="base_motor" />
-    <joint name="base_brazo" />
+    <joint name="base" />
     <mechanicalReduction>1.0</mechanicalReduction>
     <motorTorqueConstant>1.0</motorTorqueConstant>

File: MB_robot/myrabot_arm_model/urdf/brazo-macros_real.xacro (robot description, xacro)
@@ -254,5 +254,5 @@
  <transmission type="pr2_mechanism_model/SimpleTransmission" name="base_trans">
     <actuator name="base_motor" />
-    <joint name="base_brazo" />
+    <joint name="base" />
     <mechanicalReduction>1.0</mechanicalReduction>
     <motorTorqueConstant>1.0</motorTorqueConstant>

File: MB_robot/myrabot_arm_model/urdf/brazo.xacro (robot description, xacro)
@@ -31,5 +31,5 @@
     </inertial>
   </link>
-  <joint name="base_brazo" type="revolute">
+  <joint name="base" type="revolute">
     <parent link="base_brazo_link"/>
     <child link="hombro_link"/>
@@ -426,5 +426,5 @@
 <gazebo_propiedades_link nombre="pinza_link_SI" material="brazo_fer/White" />
 <gazebo_propiedades_link nombre="pinza_link_SD" material="brazo_fer/White" />
-<gazebo_propiedades_joint nombre="base_brazo" />
+<gazebo_propiedades_joint nombre="base" />
 <gazebo_propiedades_joint nombre="arti1" />
 <gazebo_propiedades_joint nombre="arti2" />

File: MB_robot/myrabot_arm_model/urdf/brazo_real.xacro (robot description, xacro)
@@ -14,9 +14,9 @@
       <origin xyz="0 0 0.019" rpy="${M_PI/2} 0 ${-M_PI/2}"/>
     </dynamixel_AX12_fixed>
-    <bioloid_F3_revolute parent="servo_base_link" name="base_brazo" color="white" vlimit="3" llimit="-2.62" ulimit="2.62">
+    <bioloid_F3_revolute parent="servo_base_link" name="base" color="white" vlimit="3" llimit="-2.62" ulimit="2.62">
       <origin xyz="0 ${AX12_WIDTH/2} 0" rpy="${-M_PI/2} ${-M_PI/2} ${-M_PI}" />
     </bioloid_F3_revolute>
     <!-- shoulder lift joint -->
-    <dynamixel_AX12_fixed parent="base_brazo_link" name="servo_arti1">
+    <dynamixel_AX12_fixed parent="base_link" name="servo_arti1">
       <origin xyz="0 0 ${-AX12_HEIGHT-F10_HEIGHT+0.001}" rpy="0 ${M_PI} 0" />
     </dynamixel_AX12_fixed>
@@ -130,5 +130,5 @@
 <gazebo_propiedades_link nombre="pinza_fija_link" material="brazo_fer/White" />
 <gazebo_propiedades_link nombre="pinza_fija_dedo_link" material="brazo_fer/WhiteTransparent" />
-<gazebo_propiedades_joint nombre="base_brazo" />
+<gazebo_propiedades_joint nombre="base" />
 <gazebo_propiedades_joint nombre="arti1" />
 <gazebo_propiedades_joint nombre="arti2" />

File: MB_robot/myrabot_robot_model/urdf/estructura-myrabot-macros.xacro (robot description, xacro)
@@ -1,4 +1,6 @@
 <?xml version="1.0"?>
 <robot xmlns:xacro="http://ros.org/wiki/xacro">
+<xacro:property name="altura_monitor" value="1.15" />
+<xacro:property name="inclinacion_monitor" value="-0.12" />
 <macro name="default_inertia_e">
 	<inertia ixx="0.05" ixy="0.0" ixz="0.0" iyy="0.05" iyz="0.0" izz="0.05"/>

File: MB_robot/myrabot_robot_model/urdf/estructura-myrabot.xacro (robot description, xacro)
@@ -332,5 +332,5 @@
   <parent link="e_pilar_link"/>
   <child link="e_soporte_1_link"/>
-  <origin xyz="0 0 ${altura_monitor-(0.708-0.115)-(0.395-0.155)}" rpy="0 0 0" />
+  <origin xyz="0 0 ${altura_monitor-(0.708-0.155)-(0.395-0.155)}" rpy="0 0 0" />
 </joint>
 <link name="e_soporte_1_link">
@@ -357,5 +357,5 @@
   <parent link="e_soporte_1_link"/>
   <child link="e_soporte_2_link"/>
-  <origin xyz="0 0.065 0.61" rpy="-${inclinacion_monitor} 0 0" />
+  <origin xyz="0 0.065 0.61" rpy="${inclinacion_monitor} 0 0" />
 </joint>
 <link name="e_soporte_2_link">
@@ -376,29 +376,4 @@
       <geometry>
         <mesh filename="package://myrabot_robot_model/meshes/e_soporte_2.stl" scale="0.001 0.001 0.001"/>
-      </geometry>
-    </collision>
-  </link>
- <joint name="soporte_3" type="fixed">
-  <parent link="e_soporte_1_link"/>
-  <child link="e_soporte_3_link"/>
-  <origin xyz="0 0.065 0.61" rpy="${-inclinacion_soporte_camara} 0 0" />
-</joint>
-<link name="e_soporte_3_link">
-    <inertial>
-      <mass value="0.01"/>
-      <origin rpy="0 0 0" xyz="0.0 -0.065 ${0.06/2}"/>
-      <default_inertia_e />
-    </inertial>
-    <visual>
-      <origin rpy="0 0 0" xyz="-0.135 -0.2 -0.03"/>
-      <geometry>
-        <mesh filename="package://myrabot_robot_model/meshes/e_soporte_3.stl" scale="0.001 0.001 0.001"/>
-      </geometry>
-      <material name="wood" />
-    </visual>
-    <collision>
-      <origin rpy="0 0 0" xyz="-0.135 -0.2 -0.03"/>
-      <geometry>
-        <mesh filename="package://myrabot_robot_model/meshes/e_soporte_3.stl" scale="0.001 0.001 0.001"/>
       </geometry>
     </collision>
@@ -478,5 +453,4 @@
 <gazebo_propiedades nombre="e_soporte_1_link" material="myrabot_fer/LightWood" />
 <gazebo_propiedades nombre="e_soporte_2_link" material="myrabot_fer/LightWood" />
-<gazebo_propiedades nombre="e_soporte_3_link" material="myrabot_fer/LightWood" />
 <gazebo_propiedades nombre="e_monitor_link" material="myrabot_fer/LightWood" />
 <gazebo_propiedades nombre="e_pantalla_link" material="myrabot_fer/Black" />

File: MB_robot/myrabot_robot_model/urdf/myrabot.urdf.xacro (robot description, xacro)
@@ -13,12 +13,4 @@
        xmlns:controller="http://playerstage.sourceforge.net/gazebo/xmlschema/#controller"
        xmlns:physics="http://playerstage.sourceforge.net/gazebo/xmlschema/#physics">
-    <!-- Propiedades estructura -->
-    <property name="altura_monitor" value="1.15" />
-	<property name="inclinacion_monitor" value="0.12" />
-	<property name="inclinacion_soporte_camara" value="-0.12" />
-    <!-- Propiedades xtion -->
-	<property name="orientacion_camara" value="0.0"/> <!-- 3.14 para cambiar orientacion camara -->
-	<property name="inclinacion_camara" value="-0.65"/> <!-- 0.0 para colocar paralela a soporte -->
-	<property name="avance_camara" value="0.03"/> <!-- 0.0 para colocar en el centro del soporte -->
 	<include filename="$(find myrabot_robot_model)/urdf/roomba.xacro" />
 	<include filename="$(find myrabot_robot_model)/urdf/estructura-myrabot.xacro" />
@@ -26,8 +18,7 @@
 	<include filename="$(find myrabot_arm_model)/urdf/brazo.xacro" />
 	<include filename="$(find myrabot_robot_model)/urdf/webcam.xacro" />
-	<!--include filename="$(find myrabot_robot_model_b)/urdf/xtion.xacro" /-->
 	<include filename="$(find myrabot_robot_model)/urdf/ultrasonidos.xacro" />
 	<roomba />
-	<estructura_myrabot parent="base_link">
+	<estructura_myrabot parent="base_roomba_link">
 		<origin rpy="0 0 1.57" xyz="0 0 0.063"/>
 	</estructura_myrabot>
@@ -38,10 +29,7 @@
 		<origin rpy="0 0 3.1416" xyz="0 -0.1015 0.075"/>
 	</brazo>
-	<webcam parent="e_soporte_3_link">
-		<origin rpy="0 0 0" xyz="-0.135 -0.135 ${0.145/2}"/>
+	<webcam parent="e_monitor_link">
+		<origin rpy="0 0 0" xyz="-0.135 -0.135 ${0.185/2}"/>
 	</webcam>
-	<!--xtion parent="e_soporte_3_link">
-		<origin rpy="0 ${-inclinacion_camara} ${-1.57+orientacion_camara}" xyz="0.0 ${-avance_camara} 0.175"/>
-	</xtion-->
 	<ultrasonidos id="1" parent="e_base_2_link" d_centro="0.150">
 		<origin rpy="0 0 1.57" xyz="0 0 ${0.04-0.007}"/>

File: MB_robot/myrabot_robot_model/urdf/myrabot_brazo_real.urdf.xacro (robot description, xacro)
@@ -13,12 +13,4 @@
        xmlns:controller="http://playerstage.sourceforge.net/gazebo/xmlschema/#controller"
        xmlns:physics="http://playerstage.sourceforge.net/gazebo/xmlschema/#physics">
-    <!-- Propiedades estructura -->
-    <property name="altura_monitor" value="1.15" />
-	<property name="inclinacion_monitor" value="0.12" />
-	<property name="inclinacion_soporte_camara" value="-0.12" />
-    <!-- Propiedades xtion -->
-	<property name="orientacion_camara" value="0.0"/> <!-- 3.14 para cambiar orientacion camara -->
-	<property name="inclinacion_camara" value="-0.65"/> <!-- 0.0 para colocar paralela a soporte -->
-	<property name="avance_camara" value="0.03"/> <!-- 0.0 para colocar en el centro del soporte -->
 	<include filename="$(find myrabot_robot_model)/urdf/roomba.xacro" />
 	<include filename="$(find myrabot_robot_model)/urdf/estructura-myrabot.xacro" />
@@ -26,8 +18,7 @@
 	<include filename="$(find myrabot_arm_model)/urdf/brazo_real.xacro" />
 	<include filename="$(find myrabot_robot_model)/urdf/webcam.xacro" />
-	<!--include filename="$(find myrabot_robot_model_b)/urdf/xtion.xacro" /-->
 	<include filename="$(find myrabot_robot_model)/urdf/ultrasonidos.xacro" />
 	<roomba />
-	<estructura_myrabot parent="base_link">
+	<estructura_myrabot parent="base_roomba_link">
 		<origin rpy="0 0 1.57" xyz="0 0 0.063"/>
 	</estructura_myrabot>
@@ -38,10 +29,7 @@
 		<origin rpy="0 0 1.57" xyz="0 -0.1015 0.075"/>
 	</brazo>
-	<webcam parent="e_soporte_3_link">
-		<origin rpy="0 0 0" xyz="-0.135 -0.135 ${0.145/2}"/>
+	<webcam parent="e_monitor_link">
+		<origin rpy="0 0 0" xyz="-0.135 -0.135 ${0.185/2}"/>
 	</webcam>
-	<!--xtion parent="e_soporte_3_link">
-		<origin rpy="0 ${-inclinacion_camara} ${-1.57+orientacion_camara}" xyz="0.0 ${-avance_camara} 0.175"/>
-	</xtion-->
 	<ultrasonidos id="1" parent="e_base_2_link" d_centro="0.150">
 		<origin rpy="0 0 1.57" xyz="0 0 ${0.04-0.007}"/>

File: MB_robot/myrabot_robot_model/urdf/roomba-gazebo.xacro (robot description, xacro)
@@ -53,5 +53,5 @@
       <wheel_separation>.230</wheel_separation>
       <wheel_diameter>0.070</wheel_diameter>
-      <base_geom>base_link</base_geom>
+      <base_geom>base_roomba_link</base_geom>
       <updateRate>40</updateRate>
       <torque>1.0</torque>

File: MB_robot/myrabot_robot_model/urdf/roomba.xacro (robot description, xacro)
@@ -4,5 +4,5 @@
   <include filename="$(find myrabot_robot_model)/urdf/roomba-gazebo.xacro"/>
 <xacro:macro name="roomba">
-  <!-- base_footprint is a fictitious link(frame) that is on the ground right below base_link origin, navigation stack depends on this frame -->
+  <!-- base_footprint is a fictitious link(frame) that is on the ground right below base_roomba_link origin, navigation stack depends on this frame -->
   <link name="base_footprint">
     <inertial>
@@ -29,5 +29,5 @@
     </collision>
   </link>
-  <link name="base_link">
+  <link name="base_roomba_link">
     <inertial>
       <mass value="3.6" />
@@ -94,29 +94,29 @@
     <origin xyz="0 0 0.017" rpy="0 0 0" />
     <parent link="base_footprint"/>
-    <child link="base_link" />
+    <child link="base_roomba_link" />
   </joint>
   <joint name="base_wall_sensor_joint" type="fixed">
     <origin xyz="0.09 -0.120 0.042" rpy="0 0 -1.0" />
-    <parent link="base_link"/>
+    <parent link="base_roomba_link"/>
     <child link="wall_sensor_link" />
   </joint>
   <joint name="base_left_cliff_sensor_joint" type="fixed">
     <origin xyz="0.07 0.14 0.01" rpy="0 1.57079 0" />
-    <parent link="base_link"/>
+    <parent link="base_roomba_link"/>
     <child link="left_cliff_sensor_link" />
   </joint>
   <joint name="base_right_cliff_sensor_joint" type="fixed">
     <origin xyz="0.07 -0.14 0.01" rpy="0 1.57079 0" />
-    <parent link="base_link"/>
+    <parent link="base_roomba_link"/>
     <child link="right_cliff_sensor_link" />
   </joint>
   <joint name="base_leftfront_cliff_sensor_joint" type="fixed">
     <origin xyz="0.15 0.04 0.01" rpy="0 1.57079 0" />
-    <parent link="base_link"/>
+    <parent link="base_roomba_link"/>
     <child link="leftfront_cliff_sensor_link" />
   </joint>
   <joint name="base_rightfront_cliff_sensor_joint" type="fixed">
     <origin xyz="0.15 -0.04 0.01" rpy="0 1.57079 0" />
-    <parent link="base_link"/>
+    <parent link="base_roomba_link"/>
     <child link="rightfront_cliff_sensor_link" />
   </joint>
@@ -143,5 +143,5 @@
   <joint name="left_wheel_joint" type="continuous">
     <origin xyz="0 0.115 0.017" rpy="0 0 0"/>
-    <parent link="base_link"/>
+    <parent link="base_roomba_link"/>
     <child link="left_wheel_link"/>
     <axis xyz="0 1 0"/>
@@ -169,5 +169,5 @@
   <joint name="right_wheel_joint" type="continuous">
     <origin xyz="0 -0.115 0.017" rpy="0 0 0"/>
-    <parent link="base_link"/>
+    <parent link="base_roomba_link"/>
     <child link="right_wheel_link"/>
     <axis xyz="0 1 0"/>
@@ -196,5 +196,5 @@
   <joint name="rear_castor_joint" type="fixed">
     <origin xyz="-0.13 0 0.0" rpy="0 0 0"/>
-    <parent link="base_link"/>
+    <parent link="base_roomba_link"/>
     <child link="rear_wheel_link"/>
     <axis xyz="0 1 0"/>
@@ -223,5 +223,5 @@
   <joint name="front_castor_joint" type="fixed">
     <origin xyz="0.13 0 0.0" rpy="0 0 0"/>
-    <parent link="base_link"/>
+    <parent link="base_roomba_link"/>
     <child link="front_wheel_link"/>
     <axis xyz="0 1 0"/>
@@ -230,5 +230,5 @@
     <axis xyz="0 1 0" />
     <origin xyz="0 0 0.04" rpy="0 0 0" />
-    <parent link="base_link"/>
+    <parent link="base_roomba_link"/>
     <child link="gyro_link"/>
   </joint>
@@ -242,5 +242,5 @@
   <joint name="laser_joint" type="fixed">
     <origin xyz="0.065 0 0.57" rpy="0 0 0" />
-    <parent link="base_link" />
+    <parent link="base_roomba_link" />
     <child link="laser" />
   </joint>
@@ -260,5 +260,5 @@
     </inertial-->
   </link>
-<gaezebo reference="base_link">
+<gaezebo reference="base_roomba_link">
   <material>myrabot_fer/White</material>
 </gaezebo>

File: MB_robot/myrabot_robot_model/urdf/webcam.xacro (robot description, xacro)
@@ -17,5 +17,5 @@
       <origin xyz=" 0 0 0 " rpy="0 0 0" />
       <geometry>
-        <mesh filename="package://myrabot_robot_model/meshes/webcam_1b.stl" scale="0.001 0.001 0.001"/>
+        <mesh filename="package://myrabot_robot_model/meshes/webcam_1.stl" scale="0.001 0.001 0.001"/>
       </geometry>
       <material name="black">
@@ -26,5 +26,5 @@
       <origin xyz="0.0 0.0 0.0" rpy="0 0 0" />
       <geometry>
-        <mesh filename="package://myrabot_robot_model/meshes/webcam_1b.stl" scale="0.001 0.001 0.001"/>
+        <mesh filename="package://myrabot_robot_model/meshes/webcam_1.stl" scale="0.001 0.001 0.001"/>
       </geometry>
     </collision>
