Commit message: Last modifications for RoCKIn Robot Challenge competition

File: MB_robot/myrabot_robot_model/urdf/xtion.xacro (robot description, xacro)
@@ -1,4 +1,4 @@
 <?xml version="1.0"?>
-<robot>
+<robot xmlns:xacro="http://ros.org/wiki/xacro">
   <!-- Xacro properties -->
   <xacro:property name="M_SCALE" value="0.001"/>
@@ -6,5 +6,6 @@
   <xacro:property name="asus_xtion_pro_cam_rel_rgb_py"   value="-0.0220" />
   <property name="M_PI" value="3.14159"/>
-  <macro name="xtion" params="parent *origin">
+  <!-- Parameterised in part by the values in turtlebot_properties.urdf.xacro -->
+  <xacro:macro name="xtion" params="parent *origin">
     <joint name="camera_rgb_joint_xtion" type="fixed">
 	  <insert_block name="origin" />
@@ -22,5 +23,5 @@
     </link>
     <joint name="camera_rgb_optical_joint_xtion" type="fixed">
-      <origin xyz="0 0 0" rpy="${-M_PI/2} 0 ${-M_PI/2}" />
+      <origin xyz="0.0175 0.022 0.021" rpy="${-M_PI/2} 0 ${-M_PI/2}" />
       <parent link="camera_rgb_frame_xtion" />
       <child link="camera_rgb_optical_frame_xtion" />
@@ -36,5 +37,5 @@
     </link>
     <joint name="camera_joint_xtion" type="fixed">
-      <origin xyz="0.0175 ${asus_xtion_pro_cam_rel_rgb_py+0.022} 0.021"
+      <origin xyz="0.0175 ${asus_xtion_pro_cam_rel_rgb_py+0.022+0.022+0.027} 0.021"
               rpy="0 0 0"/>
       <parent link="camera_rgb_frame_xtion"/>
@@ -43,13 +44,13 @@
     <link name="camera_link_xtion">
       <visual>
-        <origin xyz="-0.01 0 0" rpy="${-M_PI/2} -${M_PI} ${-M_PI/2}"/>
+        <origin xyz="-0.01 -0.049 0" rpy="${-M_PI/2} -${M_PI} ${-M_PI/2}"/>
         <geometry>
-          <mesh filename="package://myrabot_robot_model/meshes/asus_xtion_pro_live.dae" scale="${M_SCALE} ${M_SCALE} ${M_SCALE}"/>
+          <mesh filename="package://myrabot_robot_model_b/meshes/asus_xtion_pro_live.dae" scale="${M_SCALE} ${M_SCALE} ${M_SCALE}"/>
         </geometry>
       </visual>
       <collision>
-        <origin xyz="-0.01 0 0" rpy="${-M_PI/2} -${M_PI} ${-M_PI/2}"/>
+        <origin xyz="-0.01 -0.049 0" rpy="${-M_PI/2} -${M_PI} ${-M_PI/2}"/>
         <geometry>
-          <mesh filename="package://myrabot_robot_model/meshes/asus_xtion_pro_live.dae" scale="${M_SCALE} ${M_SCALE} ${M_SCALE}"/>
+          <mesh filename="package://myrabot_robot_model_b/meshes/asus_xtion_pro_live.dae" scale="${M_SCALE} ${M_SCALE} ${M_SCALE}"/>
         </geometry>
       </collision>
@@ -90,29 +91,40 @@
       </inertial>
     </link>
-  <gazebo reference="camera_link_xtion">
-    <sensor:camera name="xtion">
-      <imageFormat>R8G8B8</imageFormat>
-      <imageSize>640 480</imageSize>
-      <hfov>60</hfov>
-      <nearClip>0.05</nearClip>
-      <farClip>5</farClip>
-      <updateRate>20</updateRate>
-      <baseline>0.1</baseline>
-      <controller:gazebo_ros_openni_kinect name="kinect_camera_controller" plugin="libgazebo_ros_openni_kinect.so">
-        <alwaysOn>true</alwaysOn>
-        <updateRate>20</updateRate>
-		<robotNamespace>/</robotNamespace>
-        <imageTopicName>/xtion/image_raw</imageTopicName>
-        <pointCloudTopicName>/xtion/depth/points</pointCloudTopicName>
-        <cameraInfoTopicName>/xtion/camera_info</cameraInfoTopicName>
-        <frameName>camera_depth_optical_frame_xtion</frameName>
-        <distortion_k1>0.0</distortion_k1>
-        <distortion_k2>0.0</distortion_k2>
-        <distortion_k3>0.0</distortion_k3>
-        <distortion_t1>0.0</distortion_t1>
-        <distortion_t2>0.0</distortion_t2>
-      </controller:gazebo_ros_openni_kinect>
-    </sensor:camera>
-  </gazebo>
-  </macro>
+    <gazebo reference="camera_link_xtion">
+      <sensor type="depth" name="xtion">
+        <always_on>true</always_on>
+        <update_rate>20.0</update_rate>
+        <camera>
+          <horizontal_fov>${60.0*M_PI/180.0}</horizontal_fov>
+          <image>
+            <format>R8G8B8</format>
+            <width>640</width>
+            <height>480</height>
+          </image>
+          <clip>
+            <near>0.05</near>
+            <far>8.0</far>
+          </clip>
+        </camera>
+        <plugin name="xtion_camera_controller" filename="libgazebo_ros_openni_kinect.so">
+          <cameraName>xtion</cameraName>
+          <alwaysOn>true</alwaysOn>
+          <updateRate>10</updateRate>
+          <imageTopicName>rgb/image_raw</imageTopicName>
+          <depthImageTopicName>depth/image_raw</depthImageTopicName>
+          <pointCloudTopicName>depth/points</pointCloudTopicName>
+          <cameraInfoTopicName>rgb/camera_info</cameraInfoTopicName>
+          <depthImageCameraInfoTopicName>depth/camera_info</depthImageCameraInfoTopicName>
+          <frameName>camera_depth_optical_frame_xtion</frameName>
+          <baseline>0.1</baseline>
+          <distortion_k1>0.0</distortion_k1>
+          <distortion_k2>0.0</distortion_k2>
+          <distortion_k3>0.0</distortion_k3>
+          <distortion_t1>0.0</distortion_t1>
+          <distortion_t2>0.0</distortion_t2>
+          <pointCloudCutoff>0.4</pointCloudCutoff>
+        </plugin>
+      </sensor>
+    </gazebo>
+  </xacro:macro>
 </robot>

File: MB_robot_hydro/myrabot_robot_model_b/urdf/myrabot.urdf.xacro (robot description, xacro)
@@ -39,5 +39,5 @@
 		<origin rpy="0 0 3.1416" xyz="0 -0.1015 0.075"/>
 	</brazo>
-	<webcam parent="e_soporte_3_link">
+	<webcam parent="e_soporte_3_link" inclinacion_webcam="0.82">
 		<origin rpy="0 0 0" xyz="-0.135 -0.135 ${0.145/2}"/>
 	</webcam>

File: MB_robot_hydro/myrabot_robot_model_b/urdf/myrabot_brazo_real.urdf.xacro (robot description, xacro)
@@ -26,6 +26,6 @@
 	<xacro:include filename="$(find myrabot_robot_model_b)/urdf/kinect.xacro" />
 	<xacro:include filename="$(find myrabot_arm_model_b)/urdf/brazo_real.xacro" />
-	<!--xacro:include filename="$(find myrabot_robot_model_b)/urdf/webcam.xacro" /-->
-	<xacro:include filename="$(find myrabot_robot_model_b)/urdf/xtion.xacro" />
+	<xacro:include filename="$(find myrabot_robot_model_b)/urdf/webcam.xacro" />
+	<!--xacro:include filename="$(find myrabot_robot_model_b)/urdf/xtion.xacro" /-->
 	<xacro:include filename="$(find myrabot_robot_model_b)/urdf/ultrasonidos.xacro" />
 	<roomba />
@@ -39,10 +39,10 @@
 		<origin rpy="0 0 1.57" xyz="0 -0.1015 0.075"/>
 	</brazo>
-	<!--webcam parent="e_soporte_3_link">
+	<webcam parent="e_soporte_3_link" inclinacion_webcam="0.82">
 		<origin rpy="0 0 0" xyz="-0.135 -0.135 ${0.145/2}"/>
-	</webcam-->
-	<xtion parent="e_soporte_3_link">
+	</webcam>
+	<!--xtion parent="e_soporte_3_link">
 		<origin rpy="0 ${-inclinacion_camara} ${-1.57+orientacion_camara}" xyz="0.0 ${-avance_camara} 0.175"/>
-	</xtion>
+	</xtion-->
 	<ultrasonidos id="1" parent="e_base_2_link" d_centro="0.150">
 		<origin rpy="0 0 1.57" xyz="0 0 ${0.04-0.007}"/>

File: MB_robot_hydro/myrabot_robot_model_b/urdf/webcam.xacro (robot description, xacro)
@@ -1,5 +1,5 @@
 <?xml version="1.0"?>
 <robot xmlns:controller="http://playerstage.sourceforge.net/gazebo/xmlschema/#controller" xmlns:interface="http://playerstage.sourceforge.net/gazebo/xmlschema/#interface" xmlns:sensor="http://playerstage.sourceforge.net/gazebo/xmlschema/#sensor" xmlns:xacro="http://ros.org/wiki/xacro">
-<xacro:macro name="webcam" params="parent *origin">
+<xacro:macro name="webcam" params="parent inclinacion_webcam *origin">
   <joint name="webcam_1" type="fixed">
 	<insert_block name="origin" />
@@ -30,5 +30,5 @@
   </link>
   <joint name="webcam_2" type="fixed">
-    <origin xyz="0 ${0.135-0.04-(0.02-0.009)} ${(0.185/2)+0.0045}" rpy="0.82 0 0" />
+    <origin xyz="0 ${0.135-0.04-(0.02-0.009)} ${(0.185/2)+0.0045}" rpy="${inclinacion_webcam} 0 0" />
     <parent link="e_webcam_1_link" />
     <child link="e_webcam_2_link" />

File: MB_robot_hydro/myrabot_robot_model_b/urdf/xtion.xacro (robot description, xacro)
@@ -23,5 +23,5 @@
     </link>
     <joint name="camera_rgb_optical_joint_xtion" type="fixed">
-      <origin xyz="0 0 0" rpy="${-M_PI/2} 0 ${-M_PI/2}" />
+      <origin xyz="0.0175 0.022 0.021" rpy="${-M_PI/2} 0 ${-M_PI/2}" />
       <parent link="camera_rgb_frame_xtion" />
       <child link="camera_rgb_optical_frame_xtion" />
@@ -37,5 +37,5 @@
     </link>
     <joint name="camera_joint_xtion" type="fixed">
-      <origin xyz="0.0175 ${asus_xtion_pro_cam_rel_rgb_py+0.022} 0.021"
+      <origin xyz="0.0175 ${asus_xtion_pro_cam_rel_rgb_py+0.022+0.022+0.027} 0.021"
               rpy="0 0 0"/>
       <parent link="camera_rgb_frame_xtion"/>
@@ -44,5 +44,5 @@
     <link name="camera_link_xtion">
       <visual>
-        <origin xyz="-0.01 0 0" rpy="${-M_PI/2} -${M_PI} ${-M_PI/2}"/>
+        <origin xyz="-0.01 -0.049 0" rpy="${-M_PI/2} -${M_PI} ${-M_PI/2}"/>
         <geometry>
           <mesh filename="package://myrabot_robot_model_b/meshes/asus_xtion_pro_live.dae" scale="${M_SCALE} ${M_SCALE} ${M_SCALE}"/>
@@ -50,5 +50,5 @@
       </visual>
       <collision>
-        <origin xyz="-0.01 0 0" rpy="${-M_PI/2} -${M_PI} ${-M_PI/2}"/>
+        <origin xyz="-0.01 -0.049 0" rpy="${-M_PI/2} -${M_PI} ${-M_PI/2}"/>
         <geometry>
           <mesh filename="package://myrabot_robot_model_b/meshes/asus_xtion_pro_live.dae" scale="${M_SCALE} ${M_SCALE} ${M_SCALE}"/>
