Commit message: Modified arm model to asign the correct colors and materials

File: MB_robot_hydro/myrabot_arm_model_b/urdf/brazo-macros.xacro (robot description, xacro)
@@ -36,5 +36,5 @@
 </xacro:macro>
 <xacro:macro name="base" params="nombre">
-  <link name="${nombre}_link_B">
+  <link name="${nombre}_B_link">
 	<visual>
       <geometry>
@@ -60,5 +60,5 @@
 </xacro:macro>
 <xacro:macro name="soporte" params="nombre simetrico lado">
-  <link name="${nombre}_link_S${lado}">
+  <link name="${nombre}_S${lado}_link">
 	<visual>
       <geometry>
@@ -85,7 +85,7 @@
 <xacro:macro name="gazebo_propiedades_link" params="nombre material">
   <gazebo reference="${nombre}">
-	<mu1>100</mu1>
-	<mu2>100</mu2>
-	<kp>100000000000</kp>
+	<mu1>1</mu1>
+	<mu2>1</mu2>
+	<kp>1000000000</kp>
 	<kd>1000000000</kd>
 	<material>${material}</material>

File: MB_robot_hydro/myrabot_arm_model_b/urdf/brazo-macros_moveit.xacro (robot description, xacro)
@@ -226,7 +226,7 @@
 <xacro:macro name="gazebo_propiedades_link" params="nombre material">
   <gazebo reference="${nombre}">
-	<mu1>100</mu1>
-	<mu2>100</mu2>
-	<kp>100000000000</kp>
+	<mu1>1</mu1>
+	<mu2>1</mu2>
+	<kp>1000000000</kp>
 	<kd>1000000000</kd>
 	<material>${material}</material>

File: MB_robot_hydro/myrabot_arm_model_b/urdf/brazo-macros_real.xacro (robot description, xacro)
@@ -226,7 +226,7 @@
 <xacro:macro name="gazebo_propiedades_link" params="nombre material">
   <gazebo reference="${nombre}">
-	<mu1>100</mu1>
-	<mu2>100</mu2>
-	<kp>100000000000</kp>
+	<mu1>1</mu1>
+	<mu2>1</mu2>
+	<kp>1000000000</kp>
 	<kd>1000000000</kd>
 	<material>${material}</material>

File: MB_robot_hydro/myrabot_arm_model_b/urdf/brazo.xacro (robot description, xacro)
@@ -71,5 +71,5 @@
   <joint name="servo_arti1_B" type="fixed">
     <parent link="brazo_link"/>
-    <child link="brazo_link_B"/>
+    <child link="brazo_B_link"/>
     <origin xyz="0 0 0" rpy="0 0 0" />
 	<axis xyz="1 0 0" />
@@ -78,5 +78,5 @@
   <joint name="servo_arti1_D" type="fixed">
     <parent link="brazo_link"/>
-    <child link="brazo_link_SI"/>
+    <child link="brazo_SI_link"/>
     <origin xyz="0 0 0" rpy="0 0 0" />
 	<axis xyz="1 0 0" />
@@ -85,5 +85,5 @@
   <joint name="servo_arti1_I" type="fixed">
     <parent link="brazo_link"/>
-    <child link="brazo_link_SD"/>
+    <child link="brazo_SD_link"/>
     <origin xyz="0 0 0" rpy="0 0 0" />
 	<axis xyz="1 0 0" />
@@ -102,5 +102,5 @@
   <joint name="servo_arti2_B" type="fixed">
     <parent link="antebrazo_link"/>
-    <child link="antebrazo_link_B"/>
+    <child link="antebrazo_B_link"/>
     <origin xyz="0 0 0" rpy="0 0 0" />
 	<axis xyz="1 0 0" />
@@ -109,5 +109,5 @@
   <joint name="servo_arti2_D" type="fixed">
     <parent link="antebrazo_link"/>
-    <child link="antebrazo_link_SI"/>
+    <child link="antebrazo_SI_link"/>
     <origin xyz="0 0 0" rpy="0 0 0" />
 	<axis xyz="1 0 0" />
@@ -116,5 +116,5 @@
   <joint name="servo_arti2_I" type="fixed">
     <parent link="antebrazo_link"/>
-    <child link="antebrazo_link_SD"/>
+    <child link="antebrazo_SD_link"/>
     <origin xyz="0 0 0" rpy="0 0 0" />
 	<axis xyz="1 0 0" />
@@ -152,9 +152,9 @@
   <joint name="servo_arti3_B" type="fixed">
     <parent link="muneca_link"/>
-    <child link="muneca_link_B"/>
-    <origin xyz="0 0 0" rpy="0 0 0" />
-	<axis xyz="1 0 0" />
-  </joint>
-  <link name="muneca_link_B">
+    <child link="muneca_B_link"/>
+    <origin xyz="0 0 0" rpy="0 0 0" />
+	<axis xyz="1 0 0" />
+  </joint>
+  <link name="muneca_B_link">
 	<visual>
       <geometry>
@@ -180,9 +180,9 @@
   <joint name="servo_arti3_D" type="fixed">
     <parent link="muneca_link"/>
-    <child link="muneca_link_SI"/>
-    <origin xyz="0 0 0" rpy="0 0 0" />
-	<axis xyz="1 0 0" />
-  </joint>
-  <link name="muneca_link_SI">
+    <child link="muneca_SI_link"/>
+    <origin xyz="0 0 0" rpy="0 0 0" />
+	<axis xyz="1 0 0" />
+  </joint>
+  <link name="muneca_SI_link">
 	<visual>
       <geometry>
@@ -208,9 +208,9 @@
   <joint name="servo_arti3_I" type="fixed">
     <parent link="muneca_link"/>
-    <child link="muneca_link_SD"/>
-    <origin xyz="0 0 0" rpy="0 0 0" />
-	<axis xyz="1 0 0" />
-  </joint>
-  <link name="muneca_link_SD">
+    <child link="muneca_SD_link"/>
+    <origin xyz="0 0 0" rpy="0 0 0" />
+	<axis xyz="1 0 0" />
+  </joint>
+  <link name="muneca_SD_link">
 	<visual>
       <geometry>
@@ -236,10 +236,10 @@
   <joint name="servo_arti3_P" type="fixed">
     <parent link="muneca_link"/>
-    <child link="muneca_link_P"/>
+    <child link="muneca_P_link"/>
     <origin xyz="0 0 0" rpy="0 0 0" />
 	<axis xyz="1 0 0" />
   </joint>
   <!--pinza izquierda fija-->
-  <link name="muneca_link_P">
+  <link name="muneca_P_link">
 	<visual>
       <geometry>
@@ -265,9 +265,9 @@
   <joint name="servo_arti3_PS" type="fixed">
     <parent link="muneca_link"/>
-    <child link="muneca_link_PS"/>
-    <origin xyz="0 0 0" rpy="0 0 0" />
-	<axis xyz="1 0 0" />
-  </joint>
-  <link name="muneca_link_PS">
+    <child link="muneca_PS_link"/>
+    <origin xyz="0 0 0" rpy="0 0 0" />
+	<axis xyz="1 0 0" />
+  </joint>
+  <link name="muneca_PS_link">
 	<visual>
       <geometry>
@@ -324,9 +324,9 @@
   <joint name="servo_pinza_B" type="fixed">
     <parent link="pinza_link"/>
-    <child link="pinza_link_B"/>
-    <origin xyz="0 0 0" rpy="0 0 0" />
-	<axis xyz="1 0 0" />
-  </joint>
-  <link name="pinza_link_B">
+    <child link="pinza_B_link"/>
+    <origin xyz="0 0 0" rpy="0 0 0" />
+	<axis xyz="1 0 0" />
+  </joint>
+  <link name="pinza_B_link">
 	<visual>
       <geometry>
@@ -352,9 +352,9 @@
   <joint name="servo_pinza_D" type="fixed">
     <parent link="pinza_link"/>
-    <child link="pinza_link_SI"/>
-    <origin xyz="0 0 0" rpy="0 0 0" />
-	<axis xyz="1 0 0" />
-  </joint>
-  <link name="pinza_link_SI">
+    <child link="pinza_SI_link"/>
+    <origin xyz="0 0 0" rpy="0 0 0" />
+	<axis xyz="1 0 0" />
+  </joint>
+  <link name="pinza_SI_link">
 	<visual>
       <geometry>
@@ -380,9 +380,9 @@
   <joint name="servo_pinza_I" type="fixed">
     <parent link="pinza_link"/>
-    <child link="pinza_link_SD"/>
-    <origin xyz="0 0 0" rpy="0 0 0" />
-	<axis xyz="1 0 0" />
-  </joint>
-  <link name="pinza_link_SD">
+    <child link="pinza_SD_link"/>
+    <origin xyz="0 0 0" rpy="0 0 0" />
+	<axis xyz="1 0 0" />
+  </joint>
+  <link name="pinza_SD_link">
 	<visual>
       <geometry>
@@ -409,21 +409,21 @@
 <gazebo_propiedades_link nombre="hombro_link" material="brazo_fer/Black" />
 <gazebo_propiedades_link nombre="brazo_link" material="brazo_fer/Black" />
+<gazebo_propiedades_link nombre="brazo_B_link" material="brazo_fer/White" />
+<gazebo_propiedades_link nombre="brazo_SI_link" material="brazo_fer/White" />
+<gazebo_propiedades_link nombre="brazo_SD_link" material="brazo_fer/White" />
 <gazebo_propiedades_link nombre="antebrazo_link" material="brazo_fer/Black" />
+<gazebo_propiedades_link nombre="antebrazo_B_link" material="brazo_fer/White" />
+<gazebo_propiedades_link nombre="antebrazo_SI_link" material="brazo_fer/White" />
+<gazebo_propiedades_link nombre="antebrazo_SD_link" material="brazo_fer/White" />
 <gazebo_propiedades_link nombre="muneca_link" material="brazo_fer/Black" />
-<gazebo_propiedades_link nombre="brazo_link_B" material="brazo_fer/White" />
-<gazebo_propiedades_link nombre="brazo_link_SI" material="brazo_fer/White" />
-<gazebo_propiedades_link nombre="brazo_link_SD" material="brazo_fer/White" />
-<gazebo_propiedades_link nombre="antebrazo_link_B" material="brazo_fer/White" />
-<gazebo_propiedades_link nombre="antebrazo_link_SI" material="brazo_fer/White" />
-<gazebo_propiedades_link nombre="antebrazo_link_SD" material="brazo_fer/White" />
-<gazebo_propiedades_link nombre="muneca_link_B" material="brazo_fer/White" />
-<gazebo_propiedades_link nombre="muneca_link_SI" material="brazo_fer/White" />
-<gazebo_propiedades_link nombre="muneca_link_SD" material="brazo_fer/White" />
-<gazebo_propiedades_link nombre="muneca_link_P" material="brazo_fer/WhiteTransparent" />
-<gazebo_propiedades_link nombre="muneca_link_PS" material="brazo_fer/White" />
+<gazebo_propiedades_link nombre="muneca_B_link" material="brazo_fer/White" />
+<gazebo_propiedades_link nombre="muneca_SI_link" material="brazo_fer/White" />
+<gazebo_propiedades_link nombre="muneca_SD_link" material="brazo_fer/White" />
+<gazebo_propiedades_link nombre="muneca_P_link" material="brazo_fer/WhiteTransparent" />
+<gazebo_propiedades_link nombre="muneca_PS_link" material="brazo_fer/White" />
 <gazebo_propiedades_link nombre="pinza_link" material="brazo_fer/WhiteTransparent" />
-<gazebo_propiedades_link nombre="pinza_link_B" material="brazo_fer/White" />
-<gazebo_propiedades_link nombre="pinza_link_SI" material="brazo_fer/White" />
-<gazebo_propiedades_link nombre="pinza_link_SD" material="brazo_fer/White" />
+<gazebo_propiedades_link nombre="pinza_B_link" material="brazo_fer/White" />
+<gazebo_propiedades_link nombre="pinza_SI_link" material="brazo_fer/White" />
+<gazebo_propiedades_link nombre="pinza_SD_link" material="brazo_fer/White" />
 <gazebo_propiedades_joint nombre="base_brazo" />
 <gazebo_propiedades_joint nombre="arti1" />

File: MB_robot_hydro/myrabot_arm_model_b/urdf/brazo_moveit.xacro (robot description, xacro)
@@ -18,8 +18,8 @@
     </bioloid_F3_revolute>
     <!-- shoulder lift joint -->
-    <dynamixel_AX12_fixed parent="base_brazo_link" name="servo_arti1">
+    <dynamixel_AX12_fixed parent="base_brazo_link" name="servo_arti_1">
       <origin xyz="0 0 ${-AX12_HEIGHT-F10_HEIGHT+0.001}" rpy="0 ${M_PI} 0" />
     </dynamixel_AX12_fixed>
-    <bioloid_F4_revolute parent="servo_arti1_link" name="arti1" color="white" vlimit="3" llimit="-2.62" ulimit="2.62">
+    <bioloid_F4_revolute parent="servo_arti_1_link" name="arti1" color="white" vlimit="3" llimit="-2.62" ulimit="2.62">
       <origin xyz="0 0 0" rpy="0 0 0" />
     </bioloid_F4_revolute>
@@ -37,8 +37,8 @@
     </bioloid_F3_fixed>
     <!-- elbow joint -->
-    <dynamixel_AX12_fixed parent="arti1_F3_0_link" name="servo_arti2">
+    <dynamixel_AX12_fixed parent="arti1_F3_0_link" name="servo_arti_2">
       <origin xyz="0 0 ${-AX12_HEIGHT-F10_HEIGHT+0.001}" rpy="0 ${M_PI} 0"/>
     </dynamixel_AX12_fixed>
-    <bioloid_F4_revolute parent="servo_arti2_link" name="arti2" color="white" vlimit="3" llimit="-2.63" ulimit="2.63">
+    <bioloid_F4_revolute parent="servo_arti_2_link" name="arti2" color="white" vlimit="3" llimit="-2.63" ulimit="2.63">
       <origin xyz="0 0 0" rpy="0 0 0" />
     </bioloid_F4_revolute>
@@ -56,8 +56,8 @@
     </bioloid_F3_fixed>
     <!-- wrist joint -->
-    <dynamixel_AX12_fixed parent="arti2_F3_0_link" name="servo_arti3">
+    <dynamixel_AX12_fixed parent="arti2_F3_0_link" name="servo_arti_3">
       <origin xyz="0 0 ${-AX12_HEIGHT-F10_HEIGHT+0.001}" rpy="0 ${M_PI} 0"/>
     </dynamixel_AX12_fixed>
-    <bioloid_F2_revolute parent="servo_arti3_link" name="arti3" color="white" vlimit="3" llimit="-2.62" ulimit="2.62">
+    <bioloid_F2_revolute parent="servo_arti_3_link" name="arti3" color="white" vlimit="3" llimit="-2.62" ulimit="2.62">
       <origin xyz="0 0 0" rpy="0 0 0" />
     </bioloid_F2_revolute>
@@ -110,5 +110,5 @@
 <gazebo_propiedades_link nombre="servo_base_link" material="brazo_fer/Black" />
 <gazebo_propiedades_link nombre="base_brazo_link" material="brazo_fer/White" />
-<gazebo_propiedades_link nombre="servo_arti1_link" material="brazo_fer/Black" />
+<gazebo_propiedades_link nombre="servo_arti_1_link" material="brazo_fer/Black" />
 <gazebo_propiedades_link nombre="arti1_link" material="brazo_fer/White" />
 <gazebo_propiedades_link nombre="arti1_F10_0_link" material="brazo_fer/White" />
@@ -116,5 +116,5 @@
 <gazebo_propiedades_link nombre="arti1_F10_2_link" material="brazo_fer/White" />
 <gazebo_propiedades_link nombre="arti1_F3_0_link" material="brazo_fer/White" />
-<gazebo_propiedades_link nombre="servo_arti2_link" material="brazo_fer/Black" />
+<gazebo_propiedades_link nombre="servo_arti_2_link" material="brazo_fer/Black" />
 <gazebo_propiedades_link nombre="arti2_link" material="brazo_fer/White" />
 <gazebo_propiedades_link nombre="arti2_F10_0_link" material="brazo_fer/White" />
@@ -122,5 +122,5 @@
 <gazebo_propiedades_link nombre="arti2_F10_2_link" material="brazo_fer/White" />
 <gazebo_propiedades_link nombre="arti2_F3_0_link" material="brazo_fer/White" />
-<gazebo_propiedades_link nombre="servo_arti3_link" material="brazo_fer/Black" />
+<gazebo_propiedades_link nombre="servo_arti_3_link" material="brazo_fer/Black" />
 <gazebo_propiedades_link nombre="arti3_link" material="brazo_fer/White" />
 <gazebo_propiedades_link nombre="arti3_F3_0_link" material="brazo_fer/White" />

File: MB_robot_hydro/myrabot_arm_model_b/urdf/brazo_real.xacro (robot description, xacro)
@@ -18,8 +18,8 @@
     </bioloid_F3_revolute>
     <!-- shoulder lift joint -->
-    <dynamixel_AX12_fixed parent="base_brazo_link" name="servo_arti1">
+    <dynamixel_AX12_fixed parent="base_brazo_link" name="servo_arti_1">
       <origin xyz="0 0 ${-AX12_HEIGHT-F10_HEIGHT+0.001}" rpy="0 ${M_PI} 0" />
     </dynamixel_AX12_fixed>
-    <bioloid_F4_revolute parent="servo_arti1_link" name="arti1" color="white" vlimit="3" llimit="-2.62" ulimit="2.62">
+    <bioloid_F4_revolute parent="servo_arti_1_link" name="arti1" color="white" vlimit="3" llimit="-2.62" ulimit="2.62">
       <origin xyz="0 0 0" rpy="0 0 0" />
     </bioloid_F4_revolute>
@@ -37,8 +37,8 @@
     </bioloid_F3_fixed>
     <!-- elbow joint -->
-    <dynamixel_AX12_fixed parent="arti1_F3_0_link" name="servo_arti2">
+    <dynamixel_AX12_fixed parent="arti1_F3_0_link" name="servo_arti_2">
       <origin xyz="0 0 ${-AX12_HEIGHT-F10_HEIGHT+0.001}" rpy="0 ${M_PI} 0"/>
     </dynamixel_AX12_fixed>
-    <bioloid_F4_revolute parent="servo_arti2_link" name="arti2" color="white" vlimit="3" llimit="-2.63" ulimit="2.63">
+    <bioloid_F4_revolute parent="servo_arti_2_link" name="arti2" color="white" vlimit="3" llimit="-2.63" ulimit="2.63">
       <origin xyz="0 0 0" rpy="0 0 0" />
     </bioloid_F4_revolute>
@@ -56,8 +56,8 @@
     </bioloid_F3_fixed>
     <!-- wrist joint -->
-    <dynamixel_AX12_fixed parent="arti2_F3_0_link" name="servo_arti3">
+    <dynamixel_AX12_fixed parent="arti2_F3_0_link" name="servo_arti_3">
       <origin xyz="0 0 ${-AX12_HEIGHT-F10_HEIGHT+0.001}" rpy="0 ${M_PI} 0"/>
     </dynamixel_AX12_fixed>
-    <bioloid_F2_revolute parent="servo_arti3_link" name="arti3" color="white" vlimit="3" llimit="-2.62" ulimit="2.62">
+    <bioloid_F2_revolute parent="servo_arti_3_link" name="arti3" color="white" vlimit="3" llimit="-2.62" ulimit="2.62">
       <origin xyz="0 0 0" rpy="0 0 0" />
     </bioloid_F2_revolute>
@@ -110,5 +110,5 @@
 <gazebo_propiedades_link nombre="servo_base_link" material="brazo_fer/Black" />
 <gazebo_propiedades_link nombre="base_brazo_link" material="brazo_fer/White" />
-<gazebo_propiedades_link nombre="servo_arti1_link" material="brazo_fer/Black" />
+<gazebo_propiedades_link nombre="servo_arti_1_link" material="brazo_fer/Black" />
 <gazebo_propiedades_link nombre="arti1_link" material="brazo_fer/White" />
 <gazebo_propiedades_link nombre="arti1_F10_0_link" material="brazo_fer/White" />
@@ -116,5 +116,5 @@
 <gazebo_propiedades_link nombre="arti1_F10_2_link" material="brazo_fer/White" />
 <gazebo_propiedades_link nombre="arti1_F3_0_link" material="brazo_fer/White" />
-<gazebo_propiedades_link nombre="servo_arti2_link" material="brazo_fer/Black" />
+<gazebo_propiedades_link nombre="servo_arti_2_link" material="brazo_fer/Black" />
 <gazebo_propiedades_link nombre="arti2_link" material="brazo_fer/White" />
 <gazebo_propiedades_link nombre="arti2_F10_0_link" material="brazo_fer/White" />
@@ -122,5 +122,5 @@
 <gazebo_propiedades_link nombre="arti2_F10_2_link" material="brazo_fer/White" />
 <gazebo_propiedades_link nombre="arti2_F3_0_link" material="brazo_fer/White" />
-<gazebo_propiedades_link nombre="servo_arti3_link" material="brazo_fer/Black" />
+<gazebo_propiedades_link nombre="servo_arti_3_link" material="brazo_fer/Black" />
 <gazebo_propiedades_link nombre="arti3_link" material="brazo_fer/White" />
 <gazebo_propiedades_link nombre="arti3_F3_0_link" material="brazo_fer/White" />
