Commit message: Updated hydro version

File: MB_robot_hydro/myrabot_arm_model_b/urdf/brazo-macros.xacro (robot description, xacro)
@@ -2,5 +2,5 @@
 <robot xmlns:controller="http://playerstage.sourceforge.net/gazebo/xmlschema/#controller" xmlns:xacro="http://ros.org/wiki/xacro">
 <xacro:macro name="default_inertia">
-      <inertia ixx="0.001" ixy="0.0" ixz="0.0" iyy="0.001" iyz="0.0" izz="0.001"/>
+      <inertia ixx="0.0001" ixy="0.0" ixz="0.0" iyy="0.0001" iyz="0.0" izz="0.0001"/>
 </xacro:macro>
 <xacro:macro name="default_inertia_servos">
@@ -11,5 +11,5 @@
 </xacro:macro>
 <xacro:macro name="default_dynamics">
-      <dynamics fricction="0" damping="0" />
+      <dynamics fricction="0" damping="0.5" />
 </xacro:macro>
 <xacro:macro name="servo" params="nombre">
@@ -85,19 +85,20 @@
 <xacro:macro name="gazebo_propiedades_link" params="nombre material">
   <gazebo reference="${nombre}">
-	<mu1>1</mu1>
-	<mu2>1</mu2>
-	<kp>1000000000</kp>
-	<kd>1000000000</kd>
+	<mu1>100</mu1>
+	<mu2>100</mu2>
+	<kp>1000000</kp>
+	<kd>1</kd>
 	<material>${material}</material>
-    <selfCollide>true</selfCollide>
-    <turnGravityOff>false</turnGravityOff>
+    <!--selfCollide>true</selfCollide-->
+    <gravity>true</gravity>
   </gazebo>
 </xacro:macro>
 <xacro:macro name="gazebo_propiedades_joint" params="nombre">
  <gazebo reference="${nombre}">
-    <erp>0.1</erp>
-    <stopKd value="100000000.0" />
-    <stopKp value="100000000.0" />
+    <Kd value="1000000.0" />
+    <Kp value="1.0" />
     <fudgeFactor value="0.5" />
+    <implicitSpringDamper value="true" />
+    <provideFeedback value="true" />
  </gazebo>
 </xacro:macro>
@@ -111,6 +112,6 @@
     <joint name="base_brazo"/>
     <actuator name="base_motor">
-      <hardwareInterface>PositionJointInterface</hardwareInterface>
-      <mechanicalReduction>1</mechanicalReduction>
+      <hardwareInterface>EffortJointInterface</hardwareInterface>
+      <mechanicalReduction>250</mechanicalReduction>
     </actuator>
   </transmission>
@@ -119,6 +120,6 @@
     <joint name="arti1"/>
     <actuator name="arti1_motor">
-      <hardwareInterface>PositionJointInterface</hardwareInterface>
-      <mechanicalReduction>1</mechanicalReduction>
+      <hardwareInterface>EffortJointInterface</hardwareInterface>
+      <mechanicalReduction>250</mechanicalReduction>
     </actuator>
   </transmission>
@@ -127,6 +128,6 @@
     <joint name="arti2"/>
     <actuator name="arti3_motor">
-      <hardwareInterface>PositionJointInterface</hardwareInterface>
-      <mechanicalReduction>1</mechanicalReduction>
+      <hardwareInterface>EffortJointInterface</hardwareInterface>
+      <mechanicalReduction>250</mechanicalReduction>
     </actuator>
   </transmission>
@@ -135,6 +136,6 @@
     <joint name="arti3"/>
     <actuator name="arti3_motor">
-      <hardwareInterface>PositionJointInterface</hardwareInterface>
-      <mechanicalReduction>1</mechanicalReduction>
+      <hardwareInterface>EffortJointInterface</hardwareInterface>
+      <mechanicalReduction>250</mechanicalReduction>
     </actuator>
   </transmission>
@@ -143,6 +144,6 @@
     <joint name="pinza"/>
     <actuator name="pinza_motor">
-      <hardwareInterface>PositionJointInterface</hardwareInterface>
-      <mechanicalReduction>1</mechanicalReduction>
+      <hardwareInterface>EffortJointInterface</hardwareInterface>
+      <mechanicalReduction>250</mechanicalReduction>
     </actuator>
   </transmission>

File: MB_robot_hydro/myrabot_arm_model_b/urdf/brazo-macros_moveit.xacro (robot description, xacro)
@@ -16,5 +16,5 @@
   </material>
 <xacro:macro name="default_inertia">
-      <inertia ixx="0.001" ixy="0.0" ixz="0.0" iyy="0.001" iyz="0.0" izz="0.001"/>
+      <inertia ixx="0.0001" ixy="0.0" ixz="0.0" iyy="0.0001" iyz="0.0" izz="0.0001"/>
 </xacro:macro>
 <xacro:macro name="default_inertia_servos">
@@ -22,5 +22,5 @@
 </xacro:macro>
 <xacro:macro name="default_dynamics">
-      <dynamics fricction="0" damping="0" />
+      <dynamics fricction="0" damping="0.5" />
 </xacro:macro>
   <xacro:macro name="bioloid_F10_fixed" params="parent name color *origin">
@@ -226,19 +226,20 @@
 <xacro:macro name="gazebo_propiedades_link" params="nombre material">
   <gazebo reference="${nombre}">
-	<mu1>1</mu1>
-	<mu2>1</mu2>
-	<kp>1000000000</kp>
-	<kd>1000000000</kd>
+	<mu1>100</mu1>
+	<mu2>100</mu2>
+	<kp>1000000</kp>
+	<kd>1</kd>
 	<material>${material}</material>
-    <selfCollide>true</selfCollide>
-    <turnGravityOff>false</turnGravityOff>
+    <!--selfCollide>true</selfCollide-->
+    <gravity>true</gravity>
   </gazebo>
 </xacro:macro>
 <xacro:macro name="gazebo_propiedades_joint" params="nombre">
  <gazebo reference="${nombre}">
-    <erp>0.1</erp>
-    <stopKd value="100000000.0" />
-    <stopKp value="100000000.0" />
+    <Kd value="1000000.0" />
+    <Kp value="1.0" />
     <fudgeFactor value="0.5" />
+    <implicitSpringDamper value="true" />
+    <provideFeedback value="true" />
  </gazebo>
 </xacro:macro>
@@ -252,5 +253,5 @@
     <actuator name="base_motor">
       <hardwareInterface>EffortJointInterface</hardwareInterface>
-      <mechanicalReduction>1</mechanicalReduction>
+      <mechanicalReduction>250</mechanicalReduction>
     </actuator>
   </transmission>
@@ -260,5 +261,5 @@
     <actuator name="arti1_motor">
       <hardwareInterface>EffortJointInterface</hardwareInterface>
-      <mechanicalReduction>1</mechanicalReduction>
+      <mechanicalReduction>250</mechanicalReduction>
     </actuator>
   </transmission>
@@ -268,5 +269,5 @@
     <actuator name="arti3_motor">
       <hardwareInterface>EffortJointInterface</hardwareInterface>
-      <mechanicalReduction>1</mechanicalReduction>
+      <mechanicalReduction>250</mechanicalReduction>
     </actuator>
   </transmission>
@@ -276,5 +277,5 @@
     <actuator name="arti3_motor">
       <hardwareInterface>EffortJointInterface</hardwareInterface>
-      <mechanicalReduction>1</mechanicalReduction>
+      <mechanicalReduction>250</mechanicalReduction>
     </actuator>
   </transmission>
@@ -283,6 +284,6 @@
     <joint name="pinza"/>
     <actuator name="pinza_motor">
-      <hardwareInterface>PositionJointInterface</hardwareInterface>
-      <mechanicalReduction>1</mechanicalReduction>
+      <hardwareInterface>EffortJointInterface</hardwareInterface>
+      <mechanicalReduction>250</mechanicalReduction>
     </actuator>
   </transmission>

File: MB_robot_hydro/myrabot_arm_model_b/urdf/brazo-macros_real.xacro (robot description, xacro)
@@ -9,4 +9,5 @@
   <property name="AX12_WIDTH" value="0.038"/>
   <property name="F2_HEIGHT" value="0.0265"/>
+  <property name="HOLES_DISTANCE" value="0.00813"/>
   <material name="white">
     <color rgba="0.87 0.90 0.87 1.0"/>
@@ -16,5 +17,5 @@
   </material>
 <xacro:macro name="default_inertia">
-      <inertia ixx="0.001" ixy="0.0" ixz="0.0" iyy="0.001" iyz="0.0" izz="0.001"/>
+      <inertia ixx="0.0001" ixy="0.0" ixz="0.0" iyy="0.0001" iyz="0.0" izz="0.0001"/>
 </xacro:macro>
 <xacro:macro name="default_inertia_servos">
@@ -22,5 +23,5 @@
 </xacro:macro>
 <xacro:macro name="default_dynamics">
-      <dynamics fricction="0" damping="0" />
+      <dynamics fricction="0" damping="0.5" />
 </xacro:macro>
   <xacro:macro name="bioloid_F10_fixed" params="parent name color *origin">
@@ -76,4 +77,31 @@
           <!--mesh filename="package://myrabot_arm_model_b/meshes/finger.stl" scale="${M_SCALE} ${M_SCALE} ${M_SCALE}"/-->
           <box size="0.0865 0.038 0.002" />
+        </geometry>
+      </collision>
+    </link>
+  </xacro:macro>
+  <xacro:macro name="dedo_fixed" params="parent name color *origin">
+    <joint name="${name}_joint" type="fixed">
+      <insert_block name="origin" />
+      <parent link="${parent}"/>
+      <child link="${name}_link" />
+    </joint>
+    <link name="${name}_link">
+      <inertial>
+        <mass value="0.001" />
+        <origin xyz="0 0 0" />
+		<default_inertia/>
+      </inertial>
+      <visual>
+        <origin xyz=" 0.0 0.0 0.0 " rpy="0 0 0" />
+        <geometry>
+          <mesh filename="package://myrabot_arm_model_b/meshes/dedo.stl" scale="${M_SCALE} ${M_SCALE} ${M_SCALE}"/>
+        </geometry>
+        <material name="${color}"/>
+      </visual>
+      <collision>
+        <origin xyz=" 0.0 0.0 0.0 " rpy="0 0 0" />
+        <geometry>
+          <mesh filename="package://myrabot_arm_model_b/meshes/dedo.stl" scale="${M_SCALE} ${M_SCALE} ${M_SCALE}"/>
         </geometry>
       </collision>
@@ -226,19 +254,20 @@
 <xacro:macro name="gazebo_propiedades_link" params="nombre material">
   <gazebo reference="${nombre}">
-	<mu1>1</mu1>
-	<mu2>1</mu2>
-	<kp>1000000000</kp>
-	<kd>1000000000</kd>
+	<mu1>100</mu1>
+	<mu2>100</mu2>
+	<kp>1000000</kp>
+	<kd>1</kd>
 	<material>${material}</material>
-    <selfCollide>true</selfCollide>
-    <turnGravityOff>false</turnGravityOff>
+    <!--selfCollide>true</selfCollide-->
+    <gravity>true</gravity>
   </gazebo>
 </xacro:macro>
 <xacro:macro name="gazebo_propiedades_joint" params="nombre">
  <gazebo reference="${nombre}">
-    <erp>0.1</erp>
-    <stopKd value="100000000.0" />
-    <stopKp value="100000000.0" />
+    <Kd value="1000000.0" />
+    <Kp value="1.0" />
     <fudgeFactor value="0.5" />
+    <implicitSpringDamper value="true" />
+    <provideFeedback value="true" />
  </gazebo>
 </xacro:macro>
@@ -252,6 +281,7 @@
     <joint name="base_brazo"/>
     <actuator name="base_motor">
-      <hardwareInterface>PositionJointInterface</hardwareInterface>
-      <mechanicalReduction>1</mechanicalReduction>
+      <hardwareInterface>EffortJointInterface</hardwareInterface>
+      <mechanicalReduction>250</mechanicalReduction>
+      <motorTorqueConstant>1</motorTorqueConstant>
     </actuator>
   </transmission>
@@ -260,6 +290,7 @@
     <joint name="arti1"/>
     <actuator name="arti1_motor">
-      <hardwareInterface>PositionJointInterface</hardwareInterface>
-      <mechanicalReduction>1</mechanicalReduction>
+      <hardwareInterface>EffortJointInterface</hardwareInterface>
+      <mechanicalReduction>250</mechanicalReduction>
+      <motorTorqueConstant>1</motorTorqueConstant>
     </actuator>
   </transmission>
@@ -268,6 +299,7 @@
     <joint name="arti2"/>
     <actuator name="arti3_motor">
-      <hardwareInterface>PositionJointInterface</hardwareInterface>
-      <mechanicalReduction>1</mechanicalReduction>
+      <hardwareInterface>EffortJointInterface</hardwareInterface>
+      <mechanicalReduction>250</mechanicalReduction>
+      <motorTorqueConstant>1</motorTorqueConstant>
     </actuator>
   </transmission>
@@ -276,6 +308,7 @@
     <joint name="arti3"/>
     <actuator name="arti3_motor">
-      <hardwareInterface>PositionJointInterface</hardwareInterface>
-      <mechanicalReduction>1</mechanicalReduction>
+      <hardwareInterface>EffortJointInterface</hardwareInterface>
+      <mechanicalReduction>250</mechanicalReduction>
+      <motorTorqueConstant>1</motorTorqueConstant>
     </actuator>
   </transmission>
@@ -284,6 +317,7 @@
     <joint name="pinza"/>
     <actuator name="pinza_motor">
-      <hardwareInterface>PositionJointInterface</hardwareInterface>
-      <mechanicalReduction>1</mechanicalReduction>
+      <hardwareInterface>EffortJointInterface</hardwareInterface>
+      <mechanicalReduction>250</mechanicalReduction>
+      <motorTorqueConstant>1</motorTorqueConstant>
     </actuator>
   </transmission>

File: MB_robot_hydro/myrabot_arm_model_b/urdf/brazo_real.xacro (robot description, xacro)
@@ -62,50 +62,4 @@
       <origin xyz="0 0 0" rpy="0 0 0" />
     </bioloid_F2_revolute>
-    <bioloid_F3_fixed parent="arti3_link" name="arti3_F3_0" color="white">
-      <origin xyz="0 0.016 ${F2_HEIGHT}" rpy="0 ${M_PI} ${-M_PI/2}" />
-    </bioloid_F3_fixed>
-    <!-- gripper joint -->
-    <dynamixel_AX12_fixed parent="arti3_F3_0_link" name="servo_pinza">
-      <origin xyz="-0.02275 0 ${-AX12_WIDTH/2}" rpy="${M_PI} ${M_PI/2} 0"/>
-    </dynamixel_AX12_fixed>
-    <!-- finger 1 -->
-    <joint name="pinza" type="revolute">
-      <origin xyz="0 0 0" rpy="0 0 0"/>
-      <axis xyz="0 1 0"/>
-      <limit effort="100" velocity="3" lower="-2.62" upper="2.62" />
-      <default_dynamics/>
-      <parent link="servo_pinza_link"/>
-      <child link="pinza_movil_link" />
-    </joint>
-    <link name="pinza_movil_link">
-      <inertial>
-        <mass value="0.001" />
-        <origin xyz="0 0 0" />
-        <default_inertia/>
-      </inertial>
-      <visual>
-        <origin xyz=" 0 0 0 " rpy="0 0 0" />
-        <geometry>
-          <mesh filename="package://myrabot_arm_model_b/meshes/F2.stl" scale="${M_SCALE} ${M_SCALE} ${M_SCALE}"/>
-        </geometry>
-        <material name="white"/>
-      </visual>
-      <collision>
-        <origin xyz=" 0 0 0 " rpy="0 0 0" />
-        <geometry>
-          <mesh filename="package://myrabot_arm_model_b/meshes/F2.stl" scale="${M_SCALE} ${M_SCALE} ${M_SCALE}"/>
-        </geometry>
-      </collision>
-    </link>
-    <finger_fixed parent="pinza_movil_link" name="pinza_movil_dedo" color="white">
-      <origin xyz="0 0 ${F2_HEIGHT}" rpy="0 0 0" />
-    </finger_fixed>
-    <!-- finger 2 -->
-    <bioloid_F3_fixed parent="servo_pinza_link" name="pinza_fija" color="white">
-      <origin xyz="0 0 ${-AX12_HEIGHT-F10_HEIGHT+0.001}" rpy="0 ${M_PI} 0" />
-    </bioloid_F3_fixed>
-    <finger_fixed parent="pinza_fija_link" name="pinza_fija_dedo" color="white">
-      <origin xyz="0 0 0" rpy="0 0 ${M_PI}" />
-    </finger_fixed>
 <gazebo_propiedades_link nombre="servo_base_link" material="brazo_fer/Black" />
 <gazebo_propiedades_link nombre="base_brazo_link" material="brazo_fer/White" />
@@ -124,15 +78,86 @@
 <gazebo_propiedades_link nombre="servo_arti_3_link" material="brazo_fer/Black" />
 <gazebo_propiedades_link nombre="arti3_link" material="brazo_fer/White" />
-<gazebo_propiedades_link nombre="arti3_F3_0_link" material="brazo_fer/White" />
-<gazebo_propiedades_link nombre="servo_pinza_link" material="brazo_fer/Black" />
-<gazebo_propiedades_link nombre="pinza_movil_link" material="brazo_fer/White" />
-<gazebo_propiedades_link nombre="pinza_movil_dedo_link" material="brazo_fer/WhiteTransparent" />
-<gazebo_propiedades_link nombre="pinza_fija_link" material="brazo_fer/White" />
-<gazebo_propiedades_link nombre="pinza_fija_dedo_link" material="brazo_fer/WhiteTransparent" />
 <gazebo_propiedades_joint nombre="base_brazo" />
 <gazebo_propiedades_joint nombre="arti1" />
 <gazebo_propiedades_joint nombre="arti2" />
 <gazebo_propiedades_joint nombre="arti3" />
-<gazebo_propiedades_joint nombre="pinza" />
 </xacro:macro>
+    <xacro:macro name="pinza">
+      <!-- F3 for finger 1-finger 2 and dedo 1 -->
+      <bioloid_F3_fixed parent="arti3_link" name="arti3_F3_0" color="white">
+        <origin xyz="0 0.016 ${F2_HEIGHT}" rpy="0 ${M_PI} ${-M_PI/2}" />
+      </bioloid_F3_fixed>
+      <!-- gripper joint for finger 1-finger 2 and dedo 1 -->
+      <dynamixel_AX12_fixed parent="arti3_F3_0_link" name="servo_pinza">
+        <origin xyz="-0.02275 0 ${-AX12_WIDTH/2}" rpy="${M_PI} ${M_PI/2} 0"/>
+      </dynamixel_AX12_fixed>
+      <!-- F2 fingers and dedos 1 -->
+      <bioloid_F2_revolute parent="servo_pinza_link" name="pinza" color="white" vlimit="3" llimit="-2.62" ulimit="2.62">
+        <origin xyz="0 0 0" rpy="0 0 0" />
+      </bioloid_F2_revolute>
+      <!-- finger 1 -->
+      <finger_fixed parent="pinza_link" name="pinza_movil_finger" color="white">
+        <origin xyz="0 0 ${F2_HEIGHT}" rpy="0 0 0" />
+      </finger_fixed>
+      <!-- finger 2 -->
+      <bioloid_F3_fixed parent="servo_pinza_link" name="pinza_fija" color="white">
+        <origin xyz="0 0 ${-AX12_HEIGHT-F10_HEIGHT+0.001}" rpy="0 ${M_PI} 0" />
+      </bioloid_F3_fixed>
+      <finger_fixed parent="pinza_fija_link" name="pinza_fija_finger" color="white">
+        <origin xyz="0 0 0" rpy="0 0 ${M_PI}" />
+      </finger_fixed>
+      <gazebo_propiedades_link nombre="arti3_F3_0_link" material="brazo_fer/White" />
+      <gazebo_propiedades_link nombre="servo_pinza_link" material="brazo_fer/Black" />
+      <gazebo_propiedades_link nombre="pinza_link" material="brazo_fer/White" />
+      <gazebo_propiedades_link nombre="pinza_movil_finger_link" material="brazo_fer/WhiteTransparent" />
+      <gazebo_propiedades_link nombre="pinza_fija_link" material="brazo_fer/White" />
+      <gazebo_propiedades_link nombre="pinza_fija_finger_link" material="brazo_fer/WhiteTransparent" />
+      <gazebo_propiedades_joint nombre="pinza" />
+    </xacro:macro>
+    <xacro:macro name="dedo_1">
+      <!-- F3 for finger 1-finger 2 and dedo 1 -->
+      <bioloid_F3_fixed parent="arti3_link" name="arti3_F3_0" color="white">
+        <origin xyz="0 0.016 ${F2_HEIGHT}" rpy="0 ${M_PI} ${-M_PI/2}" />
+      </bioloid_F3_fixed>
+      <!-- gripper joint for finger 1-finger 2 and dedo 1 -->
+      <dynamixel_AX12_fixed parent="arti3_F3_0_link" name="servo_pinza">
+        <origin xyz="-0.02275 0 ${-AX12_WIDTH/2}" rpy="${M_PI} ${M_PI/2} 0"/>
+      </dynamixel_AX12_fixed>
+      <!-- F2 fingers and dedos 1 -->
+      <bioloid_F2_revolute parent="servo_pinza_link" name="pinza" color="white" vlimit="3" llimit="-2.62" ulimit="2.62">
+        <origin xyz="0 0 0" rpy="0 0 0" />
+      </bioloid_F2_revolute>
+      <!-- dedo 1 -->
+      <dedo_fixed parent="pinza_link" name="pinza_movil_dedo" color="black">
+        <origin xyz="${-0.025/2} ${-0.038/2} ${(-0.049/2)+0.002}" rpy="0 0 0" />
+      </dedo_fixed>
+      <gazebo_propiedades_link nombre="arti3_F3_0_link" material="brazo_fer/White" />
+      <gazebo_propiedades_link nombre="servo_pinza_link" material="brazo_fer/Black" />
+      <gazebo_propiedades_link nombre="pinza_link" material="brazo_fer/White" />
+      <gazebo_propiedades_link nombre="pinza_movil_dedo_link" material="brazo_fer/Black" />
+      <gazebo_propiedades_joint nombre="pinza" />
+    </xacro:macro>
+    <xacro:macro name="dedo_2">
+      <!-- F3 for dedo 2 -->
+      <bioloid_F3_fixed parent="arti3_link" name="arti3_F3_0" color="white">
+        <origin xyz="0 ${(HOLES_DISTANCE*3) - 0.0004} ${F2_HEIGHT}" rpy="0 ${M_PI} ${-M_PI/2}" />
+      </bioloid_F3_fixed>
+      <!-- gripper joint for dedo 2 -->
+      <dynamixel_AX12_fixed parent="arti3_F3_0_link" name="servo_pinza">
+        <origin xyz="0 0 ${-AX12_HEIGHT - F3_HEIGHT/2}" rpy="0 ${M_PI} 0"/>
+      </dynamixel_AX12_fixed>
+      <!-- F2 dedo 2 -->
+      <bioloid_F2_revolute parent="servo_pinza_link" name="pinza" color="white" vlimit="3" llimit="-2.62" ulimit="2.62">
+        <origin xyz="0 0 0" rpy="0 ${M_PI/2} 0" />
+      </bioloid_F2_revolute>
+      <!-- dedo 2 -->
+      <dedo_fixed parent="pinza_link" name="pinza_movil_dedo" color="black">
+        <origin xyz="${0.025/2} ${-0.038/2} ${0.049+0.003+F2_HEIGHT}" rpy="${M_PI} 0 ${M_PI}" />
+      </dedo_fixed>
+      <gazebo_propiedades_link nombre="arti3_F3_0_link" material="brazo_fer/White" />
+      <gazebo_propiedades_link nombre="servo_pinza_link" material="brazo_fer/Black" />
+      <gazebo_propiedades_link nombre="pinza_link" material="brazo_fer/White" />
+      <gazebo_propiedades_link nombre="pinza_movil_dedo_link" material="brazo_fer/Black" />
+      <gazebo_propiedades_joint nombre="pinza" />
+    </xacro:macro>
 </robot>

File: MB_robot_hydro/myrabot_objects_models_b/urdf/lata_amstel.xacro (robot description, xacro)
@@ -85,22 +85,22 @@
 <gazebo reference="lata_link">
   <material>objetos_fer/Amstel</material>
-  <mu1>10</mu1>
-  <mu2>10</mu2>
+  <mu1>1</mu1>
+  <mu2>1</mu2>
   <selfCollide>true</selfCollide>
-  <turnGravityOff>true</turnGravityOff>
+  <gravity>true</gravity>
 </gazebo>
 <gazebo reference="lata_top_link">
   <material>objetos_fer/Grey0</material>
-  <mu1>10</mu1>
-  <mu2>10</mu2>
+  <mu1>1</mu1>
+  <mu2>1</mu2>
   <selfCollide>true</selfCollide>
-  <turnGravityOff>true</turnGravityOff>
+  <gravity>true</gravity>
 </gazebo>
 <gazebo reference="lata_bottom_link">
   <material>objetos_fer/Grey0</material>
-  <mu1>10</mu1>
-  <mu2>10</mu2>
+  <mu1>1</mu1>
+  <mu2>1</mu2>
   <selfCollide>true</selfCollide>
-  <turnGravityOff>true</turnGravityOff>
+  <gravity>true</gravity>
 </gazebo>
 </robot>

File: MB_robot_hydro/myrabot_objects_models_b/urdf/lata_coca_cola.xacro (robot description, xacro)
@@ -85,22 +85,22 @@
 <gazebo reference="lata_link">
   <material>objetos_fer/Cola</material>
-  <mu1>10</mu1>
-  <mu2>10</mu2>
+  <mu1>1</mu1>
+  <mu2>1</mu2>
   <selfCollide>true</selfCollide>
-  <turnGravityOff>true</turnGravityOff>
+  <gravity>true</gravity>
 </gazebo>
 <gazebo reference="lata_top_link">
   <material>objetos_fer/Grey0</material>
-  <mu1>10</mu1>
-  <mu2>10</mu2>
+  <mu1>1</mu1>
+  <mu2>1</mu2>
   <selfCollide>true</selfCollide>
-  <turnGravityOff>true</turnGravityOff>
+  <gravity>true</gravity>
 </gazebo>
 <gazebo reference="lata_bottom_link">
   <material>objetos_fer/Grey0</material>
-  <mu1>10</mu1>
-  <mu2>10</mu2>
+  <mu1>1</mu1>
+  <mu2>1</mu2>
   <selfCollide>true</selfCollide>
-  <turnGravityOff>true</turnGravityOff>
+  <gravity>true</gravity>
 </gazebo>
 </robot>

File: MB_robot_hydro/myrabot_objects_models_b/urdf/mesa.xacro (robot description, xacro)
@@ -27,5 +27,5 @@
     <origin rpy="0 0 0" xyz="0 0 ${(0.03/2)+altura}" />
     <mass value="5" />
-      <inertia ixx="0.1" ixy="0.0" ixz="0.0" iyy="0.1" iyz="0.0" izz="0.1"/>
+      <inertia ixx="0.25" ixy="0.0" ixz="0.0" iyy="0.25" iyz="0.0" izz="0.25"/>
   </inertial>
 </link>
@@ -65,6 +65,6 @@
 <gazebo reference="mesa_link">
   <material>objetos_fer/LightWood</material>
-  <mu1>10</mu1>
-  <mu2>10</mu2>
+  <mu1>1</mu1>
+  <mu2>1</mu2>
   <selfCollide>true</selfCollide>
   <turnGravityOff>false</turnGravityOff>
@@ -73,8 +73,8 @@
 <gazebo reference="pata_${id}_link">
   <material>objetos_fer/Black</material>
-  <mu1>0.9</mu1>
-  <mu2>0.9</mu2>
+  <mu1>1</mu1>
+  <mu2>1</mu2>
   <selfCollide>true</selfCollide>
-  <turnGravityOff>false</turnGravityOff>
+  <gravity>true</gravity>
 </gazebo>
 </xacro:macro>

File: MB_robot_hydro/myrabot_robot_model_b/urdf/estructura-myrabot-macros.xacro (robot description, xacro)
@@ -2,5 +2,5 @@
 <robot xmlns:xacro="http://ros.org/wiki/xacro">
 <xacro:macro name="default_inertia_e">
-	<inertia ixx="0.05" ixy="0.0" ixz="0.0" iyy="0.05" iyz="0.0" izz="0.05"/>
+	<inertia ixx="0.01" ixy="0.0" ixz="0.0" iyy="0.01" iyz="0.0" izz="0.01"/>
 </xacro:macro>
 <xacro:macro name="separador_base" params="id">
@@ -67,8 +67,10 @@
 <gazebo reference="${nombre}">
   <material>${material}</material>
-  <mu1>0.5</mu1>
-  <mu2>0.5</mu2>
-  <selfCollide>true</selfCollide>
-  <turnGravityOff>false</turnGravityOff>
+  <mu1>100</mu1>
+  <mu2>100</mu2>
+  <kp>1000000.0</kp>
+  <kd>1.0</kd>
+  <!--selfCollide>true</selfCollide-->
+  <gravity>true</gravity>
 </gazebo>
 </xacro:macro>
