Commit message: Updated hydro version

File: MB_robot_hydro/myrabot_robot_model_b/urdf/estructura-myrabot.xacro (robot description, xacro)
@@ -3,5 +3,5 @@
 	<xacro:include filename="$(find myrabot_robot_model_b)/urdf/estructura-myrabot-macros.xacro" />
 <xacro:macro name="estructura_myrabot" params="parent *origin">
-<joint name="world_joint" type="fixed">
+<joint name="estructura_joint" type="fixed">
   <parent link="${parent}"/>
   <child link="e_base_1_link"/>
@@ -10,7 +10,7 @@
   <link name="e_base_1_link">
     <inertial>
-      <mass value="0.08"/>
+      <mass value="2.0"/>
       <origin rpy="0 0 0" xyz="0.0 0.0 ${0.015/2}"/>
-      <default_inertia_e />
+      <inertia ixx="0.1" ixy="0.0" ixz="0.0" iyy="0.1" iyz="0.0" izz="0.1"/>
     </inertial>
     <visual>
@@ -45,7 +45,7 @@
   <link name="e_base_2_link">
     <inertial>
-      <mass value="0.08"/>
+      <mass value="2.0"/>
       <origin rpy="0 0 0" xyz="0.0 0.0 ${0.02/2}"/>
-      <default_inertia_e />
+      <inertia ixx="0.1" ixy="0.0" ixz="0.0" iyy="0.1" iyz="0.0" izz="0.1"/>
     </inertial>
     <visual>
@@ -332,5 +332,5 @@
   <parent link="e_pilar_link"/>
   <child link="e_soporte_1_link"/>
-  <origin xyz="0 0 ${altura_monitor-(0.708-0.115)-(0.395-0.115)}" rpy="0 0 0" />
+  <origin xyz="0 0 ${altura_monitor-((0.64 - 0.03) + 0.23)}" rpy="0 0 0" />
 </joint>
 <link name="e_soporte_1_link">

File: MB_robot_hydro/myrabot_robot_model_b/urdf/myrabot_brazo_real.urdf.xacro (robot description, xacro)
@@ -18,7 +18,7 @@
 	<xacro:property name="inclinacion_monitor" value="0.12" />
 	<xacro:property name="inclinacion_soporte_camara" value="-0.12" />
-    <!-- Propiedades estructura -->
+    <!-- Propiedades xtion -->
 	<xacro:property name="orientacion_camara" value="0.0"/> <!-- 3.14 para cambiar orientacion camara -->
-	<xacro:property name="inclinacion_camara" value="-0.65"/> <!-- 0.0 para colocar perpendicular a soporte -->
+	<xacro:property name="inclinacion_camara" value="-0.60"/> <!-- 0.0 para colocar perpendicular a soporte -->
 	<xacro:property name="avance_camara" value="0.03"/> <!-- 0.0 para colocar en el centro del soporte -->
 	<xacro:include filename="$(find myrabot_robot_model_b)/urdf/roomba.xacro" />
@@ -26,8 +26,37 @@
 	<xacro:include filename="$(find myrabot_robot_model_b)/urdf/kinect.xacro" />
 	<xacro:include filename="$(find myrabot_arm_model_b)/urdf/brazo_real.xacro" />
-	<xacro:include filename="$(find myrabot_robot_model_b)/urdf/webcam.xacro" />
-	<!--xacro:include filename="$(find myrabot_robot_model_b)/urdf/xtion.xacro" /-->
+	<!--xacro:include filename="$(find myrabot_robot_model_b)/urdf/webcam.xacro" /-->
+	<xacro:include filename="$(find myrabot_robot_model_b)/urdf/xtion.xacro" />
 	<xacro:include filename="$(find myrabot_robot_model_b)/urdf/ultrasonidos.xacro" />
+	<!--link name="world" />
+	<roomba parent="world" /-->
 	<roomba />
+	<!--joint name="robot_at_home_joint" type="fixed">
+	  <parent link="base_footprint"/>
+	  <child link="robot_at_home"/>
+	  <origin xyz="${0.12263 - (0.17)} 0.0075238 1.3666" rpy="0 0 0" />
+	</joint>
+  <link name="robot_at_home">
+    <inertial>
+      <mass value="0.010"/>
+      <origin rpy="0 0 0" xyz="0.0 0.0 0.0"/>
+      <inertia ixx="0.01" ixy="0.0" ixz="0.0" iyy="0.01" iyz="0.0" izz="0.01"/>
+    </inertial>
+    <visual>
+      <origin rpy="0 0 0" xyz="0.0 0.0 0.0"/>
+      <geometry>
+        <box size="0.01 0.01 0.01" />
+      </geometry>
+      <material name="grey">
+		<color rgba="0.5 0.5 0.5 1" />
+	  </material>
+    </visual>
+    <collision>
+      <origin rpy="0 0 0" xyz="0.0 0.0 0.0"/>
+      <geometry>
+        <box size="0.01 0.01 0.01" />
+      </geometry>
+    </collision>
+  </link-->
 	<estructura_myrabot parent="base_link">
 		<origin rpy="0 0 1.57" xyz="0 0 0.063"/>
@@ -39,10 +68,13 @@
 		<origin rpy="0 0 1.57" xyz="0 -0.1015 0.075"/>
 	</brazo>
-	<webcam parent="e_soporte_3_link" inclinacion_webcam="0.82">
+	<pinza />
+	<!--dedo_1 />
+	<dedo_2 /-->
+	<!--webcam parent="e_soporte_3_link" inclinacion_webcam="0.82">
 		<origin rpy="0 0 0" xyz="-0.135 -0.135 ${0.145/2}"/>
-	</webcam>
-	<!--xtion parent="e_soporte_3_link">
-		<origin rpy="0 ${-inclinacion_camara} ${-1.57+orientacion_camara}" xyz="0.0 ${-avance_camara} 0.175"/>
-	</xtion-->
+	</webcam-->
+	<xtion parent="e_soporte_3_link">
+		<origin rpy="0 ${-inclinacion_camara} ${-1.57+orientacion_camara}" xyz="0.0 ${-avance_camara} 0.180"/>
+	</xtion>
 	<ultrasonidos id="1" parent="e_base_2_link" d_centro="0.150">
 		<origin rpy="0 0 1.57" xyz="0 0 ${0.04-0.007}"/>

File: MB_robot_hydro/myrabot_robot_model_b/urdf/roomba-gazebo.xacro (robot description, xacro)
@@ -2,8 +2,8 @@
 <robot xmlns:controller="http://playerstage.sourceforge.net/gazebo/xmlschema/#controller" xmlns:interface="http://playerstage.sourceforge.net/gazebo/xmlschema/#interface" xmlns:sensor="http://playerstage.sourceforge.net/gazebo/xmlschema/#sensor" xmlns:xacro="http://ros.org/wiki/xacro">
 	<xacro:macro name="myrabot_sim_roomba">
-<gazebo>
+<!--gazebo>
   <plugin name="roomba_controller" filename="libgazebo_ros_create.so">
 	      <alwaysOn>true</alwaysOn>
-	      <node_namespace>myrabot_node</node_namespace>
+	      <node_namespace>/</node_namespace>
 	      <left_wheel_joint>left_wheel_joint</left_wheel_joint>
 	      <right_wheel_joint>right_wheel_joint</right_wheel_joint>
@@ -16,45 +16,71 @@
 	      <torque>10.0</torque>
   </plugin>
-</gazebo>
-<!--gazebo>
+</gazebo-->
+<gazebo>
   <plugin name="differential_drive_controller" filename="libgazebo_ros_diff_drive.so">
     <alwaysOn>true</alwaysOn>
+    <rosDebugLevel>na</rosDebugLevel>
     <updateRate>40</updateRate>
-    <leftJoint>left_wheel_joint</leftJoint>
-    <rightJoint>right_wheel_joint</rightJoint>
+    <leftJoint>right_wheel_joint</leftJoint>
+    <rightJoint>left_wheel_joint</rightJoint>
     <wheelSeparation>0.23</wheelSeparation>
     <wheelDiameter>0.07</wheelDiameter>
-    <torque>20</torque>
+    <publishWheelTF>false</publishWheelTF>
+    <wheelAcceleration>0</wheelAcceleration>
+    <wheelTorque>5</wheelTorque>
     <commandTopic>cmd_vel</commandTopic>
+    <odometrySource>world</odometrySource>
     <odometryTopic>odom</odometryTopic>
     <odometryFrame>odom</odometryFrame>
     <robotBaseFrame>base_footprint</robotBaseFrame>
+    <publishWheelJointState>true</publishWheelJointState>
+    <publishTf>1</publishTf>
   </plugin>
-</gazebo-->
+</gazebo>
+    <transmission name="right_wheel_joint_trans">
+      <type>transmission_interface/SimpleTransmission</type>
+      <joint name="right_wheel_joint">
+      </joint>
+      <actuator name="right_wheel_joint_motor">
+		<hardwareInterface>EffortJointInterface</hardwareInterface>
+        <mechanicalReduction>250</mechanicalReduction>
+      </actuator>
+    </transmission>
+    <transmission name="left_wheel_joint_trans">
+      <type>transmission_interface/SimpleTransmission</type>
+      <joint name="left_wheel_joint">
+      </joint>
+      <actuator name="left_wheel_joint_motor">
+		<hardwareInterface>EffortJointInterface</hardwareInterface>
+        <mechanicalReduction>250</mechanicalReduction>
+      </actuator>
+    </transmission>
     <gazebo reference="left_wheel_link">
       <mu1 value="100"/>
       <mu2 value="100"/>
-      <kp value="100000000.0"/>
-      <kd value="10000.0"/>
-      <!--fdir1 value="0.1 0 0"/-->
+      <kp value="1000000.0"/>
+      <kd value="1.0"/>
+      <!--fdir1 value="0 1 0"/-->
     </gazebo>
     <gazebo reference="right_wheel_link">
       <mu1 value="100"/>
       <mu2 value="100"/>
-      <kp value="100000000.0"/>
-      <kd value="10000.0"/>
-      <!--fdir1 value="0.1 0 0"/-->
+      <kp value="1000000.0"/>
+      <kd value="1.0"/>
+      <!--fdir1 value="0 1 0"/-->
     </gazebo>
     <gazebo reference="rear_wheel_link">
       <mu1 value="0"/>
       <mu2 value="0"/>
-      <kp value="100000000.0"/>
-      <kd value="10000.0"/>
+      <kp value="1000000.0"/>
+      <kd value="1.0"/>
+      <!--fdir1 value="0 1 0"/-->
     </gazebo>
     <gazebo reference="front_wheel_link">
       <mu1 value="0"/>
       <mu2 value="0"/>
-      <kp value="100000000.0"/>
-      <kd value="10000.0"/>
+      <kp value="1000000.0"/>
+      <kd value="1.0"/>
+      <!--fdir1 value="0 1 0"/-->
     </gazebo>
 	</xacro:macro>

File: MB_robot_hydro/myrabot_robot_model_b/urdf/roomba.xacro (robot description, xacro)
@@ -5,33 +5,16 @@
 <xacro:macro name="roomba">
   <!-- base_footprint is a fictitious link(frame) that is on the ground right below base_link origin, navigation stack depends on this frame -->
-  <link name="base_footprint">
-    <inertial>
-      <mass value="0.0001" />
-      <origin xyz="0 0 0" />
-      <inertia ixx="0.0001" ixy="0.0" ixz="0.0"
-              iyy="0.0001" iyz="0.0"
-              izz="0.0001" />
-    </inertial>
-    <visual>
-      <origin xyz="0 0 0" rpy="0 0 0" />
-      <geometry>
-        <box size="0.001 0.001 0.001" />
-      </geometry>
-		<material name="Green">
-		  <color rgba="0.0 0.8 0.0 1.0"/>
-		</material>
-    </visual>
-    <collision>
-      <origin xyz="0 0 0.017" rpy="0 0 0" />
-      <geometry>
-       <box size="0.001 0.001 0.001" />
-      </geometry>
-    </collision>
-  </link>
+<!--xacro:macro name="roomba" params="parent">
+  <joint name="world_joint" type="fixed">
+    <origin xyz="0 0 0" rpy="0 0 0" />
+    <parent link="${parent}"/>
+    <child link="base_footprint" />
+  </joint-->
+  <link name="base_footprint"/>
   <link name="base_link">
     <inertial>
       <mass value="3.6" />
       <origin xyz="0 0 ${0.063/2}" />
-      <inertia ixx="1" ixy="0.0" ixz="0.0" iyy="1" iyz="0.0" izz="1" />
+      <inertia ixx="0.1" ixy="0.0" ixz="0.0" iyy="0.1" iyz="0.0" izz="0.1" />
     </inertial>
     <visual>
@@ -124,7 +107,7 @@
     <inertial>
       <origin xyz="0 0 0"/>
-      <mass value="0.01" />
-      <inertia ixx="0.001" ixy="0.0" ixz="0.0"
-        iyy="0.001" iyz="0.0" izz="0.001" />
+      <mass value="0.15" />
+      <inertia ixx="0.01" ixy="0.0" ixz="0.0"
+        iyy="0.01" iyz="0.0" izz="0.01" />
     </inertial>
     <visual>
@@ -142,5 +125,5 @@
   </link>
   <joint name="left_wheel_joint" type="continuous">
-    <origin xyz="0 0.115 0.017" rpy="0 0 0"/>
+    <origin xyz="0 0.115 0.018" rpy="0 0 0"/>
     <parent link="base_link"/>
     <child link="left_wheel_link"/>
@@ -150,7 +133,7 @@
     <inertial>
       <origin xyz="0 0 0"/>
-      <mass value="0.01" />
-      <inertia ixx="0.001" ixy="0.0" ixz="0.0"
-        iyy="0.001" iyz="0.0" izz="0.001" />
+      <mass value="0.15" />
+      <inertia ixx="0.01" ixy="0.0" ixz="0.0"
+        iyy="0.01" iyz="0.0" izz="0.01" />
     </inertial>
     <visual>
@@ -168,5 +151,5 @@
   </link>
   <joint name="right_wheel_joint" type="continuous">
-    <origin xyz="0 -0.115 0.017" rpy="0 0 0"/>
+    <origin xyz="0 -0.115 0.018" rpy="0 0 0"/>
     <parent link="base_link"/>
     <child link="right_wheel_link"/>
@@ -183,11 +166,11 @@
       <origin xyz="0 0 0" rpy="0 1.5707 1.5707"/>
       <geometry>
-        <sphere radius="0.017" />
-      </geometry>
-    </visual>
-    <collision>
-      <origin xyz="0 0 0" rpy="0 1.5707 1.5707" />
-      <geometry>
-        <sphere radius="0.017" />
+        <cylinder radius="0.017" length="0.017" />
+      </geometry>
+    </visual>
+    <collision>
+      <origin xyz="0 0 0" rpy="0 1.5707 1.5707" />
+      <geometry>
+        <cylinder radius="0.017" length="0.017" />
       </geometry>
     </collision>
@@ -210,11 +193,11 @@
       <origin xyz="0 0 0" rpy="0 1.5707 1.5707"/>
       <geometry>
-        <sphere radius="0.017" />
-      </geometry>
-    </visual>
-    <collision>
-      <origin xyz="0 0 0" rpy="0 1.5707 1.5707" />
-      <geometry>
-        <sphere radius="0.017" />
+        <cylinder radius="0.017" length="0.017" />
+      </geometry>
+    </visual>
+    <collision>
+      <origin xyz="0 0 0" rpy="0 1.5707 1.5707" />
+      <geometry>
+        <cylinder radius="0.017" length="0.017" />
       </geometry>
     </collision>
@@ -245,19 +228,5 @@
     <child link="laser" />
   </joint>
-  <link name="laser">
-    <!--visual>
-      <geometry>
-        <box size="0.02 0.035 0.002" />
-      </geometry>
-      <material name="Green" />
-    </visual>
-    <inertial>
-      <mass value="0.001" />
-      <origin xyz="0 0 0" />
-      <inertia ixx="0.0001" ixy="0.0" ixz="0.0"
-        iyy="0.0001" iyz="0.0"
-        izz="0.0001" />
-    </inertial-->
-  </link>
+  <link name="laser"/>
 <gaezebo reference="base_link">
   <material>myrabot_fer/White</material>

File: MB_robot_hydro/myrabot_robot_model_b/urdf/ultrasonidos.xacro (robot description, xacro)
@@ -38,7 +38,7 @@
 <gazebo reference="ultrasonidos_${id}_link_fisico">
   <material>myrabot_fer/Black</material>
-  <mu1>0.5</mu1>
-  <mu2>0.5</mu2>
-  <selfCollide>true</selfCollide>
+  <mu1>100</mu1>
+  <mu2>100</mu2>
+  <!--selfCollide>true</selfCollide-->
   <turnGravityOff>false</turnGravityOff>
 </gazebo>

File: MB_robot_hydro/myrabot_robot_model_b/urdf/webcam.xacro (robot description, xacro)
@@ -83,21 +83,21 @@
 <gazebo reference="e_webcam_1_link">
   <material>myrabot_fer/Black</material>
-  <mu1>0.5</mu1>
-  <mu2>0.5</mu2>
-  <selfCollide>true</selfCollide>
+  <mu1>100</mu1>
+  <mu2>100</mu2>
+  <!--selfCollide>true</selfCollide-->
   <turnGravityOff>false</turnGravityOff>
 </gazebo>
 <gazebo reference="e_webcam_2_link">
   <material>myrabot_fer/Black</material>
-  <mu1>0.5</mu1>
-  <mu2>0.5</mu2>
-  <selfCollide>true</selfCollide>
+  <mu1>100</mu1>
+  <mu2>100</mu2>
+  <!--selfCollide>true</selfCollide-->
   <turnGravityOff>false</turnGravityOff>
 </gazebo>
 <gazebo reference="e_webcam_optica_link">
   <material>myrabot_fer/White</material>
-  <mu1>0.5</mu1>
-  <mu2>0.5</mu2>
-  <selfCollide>true</selfCollide>
+  <mu1>100</mu1>
+  <mu2>100</mu2>
+  <!--selfCollide>true</selfCollide-->
   <turnGravityOff>false</turnGravityOff>
 </gazebo>
